File: breakout.brd (EAGLE design)
At the start: 50 x 50 mm, 15 parts

Commit message: Routing and gerbers
Parts:
- added C1, C2, C3, C4: (no value), PN_default:0603
- added CON13, CON14, CON15, CON16, CON18, CON19, CON20, CON21: (no value), us_obudowy:PIN8X1_SM50
- added CON17, CON22: (no value), pins:PIN3X1
- added IC2: (no value), us_obudowy:MLF32-TH
- added IC3: (no value), us_obudowy:TQFP32
- added US1, US2: (no value), semiconductors:SO08
- moved CON5 26.7 mm to (29.8, 38.7)
- moved CON7 26.7 mm to (47.6, 38.7)
- moved CON8 26.7 mm to (38.7, 47.6)
- moved U$1 26.7 mm to (38.7, 38.7)
- moved CON6 26.7 mm to (38.7, 29.8)
- moved CON1 3.42 mm to (2.54, 9.53)
- moved CON2 3.42 mm to (9.53, 2.54)
- moved CON4 3.42 mm to (9.53, 16.5)
- moved IC1 3.42 mm to (9.53, 9.53)
- moved CON3 3.42 mm to (16.5, 9.53)
- moved CON11 2.93 mm to (25.7, 35.6)
- moved CON10 2.62 mm to (14.0, 23.5)
- moved CON12 2.62 mm to (14.0, 47.6)
- moved U$2 2.62 mm to (14.0, 35.6)
- moved CON9 2.31 mm to (2.22, 35.6)
Connections:
- new net N$141: CON13.P$1, IC2.1
- new net N$142: CON13.P$2, IC2.2
- new net N$143: CON13.P$3, IC2.3
- new net N$144: CON13.P$4, IC2.4
- new net N$145: CON13.P$5, IC2.5
- new net N$146: CON13.P$6, IC2.6
- new net N$147: CON13.P$7, IC2.7
- new net N$148: CON13.P$8, IC2.8
- new net N$149: CON14.P$1, IC2.9
- new net N$150: CON14.P$2, IC2.10
- new net N$151: CON14.P$3, IC2.11
- new net N$152: CON14.P$4, IC2.12
- new net N$153: CON14.P$5, IC2.13
- new net N$154: CON14.P$6, IC2.14
- new net N$155: CON14.P$7, IC2.15
- new net N$156: CON14.P$8, IC2.16
- new net N$157: CON15.P$1, IC2.17
- new net N$158: CON15.P$2, IC2.18
- new net N$159: CON15.P$3, IC2.19
- new net N$160: CON15.P$4, IC2.20
- new net N$161: CON15.P$5, IC2.21
- new net N$162: CON15.P$6, IC2.22
- new net N$163: CON15.P$7, IC2.23
- new net N$164: CON15.P$8, IC2.24
- new net N$165: CON16.P$1, IC2.25
- new net N$166: CON16.P$2, IC2.26
- new net N$167: CON16.P$3, IC2.27
- new net N$168: CON16.P$4, IC2.28
- new net N$169: CON16.P$5, IC2.29
- new net N$170: CON16.P$6, IC2.30
- new net N$171: CON16.P$7, IC2.31
- new net N$172: CON16.P$8, IC2.32
- new net N$177: C2.1, CON17.1, US1.1
- new net N$178: C1.1, CON17.3, US1.8
- new net N$179: C1.2, C2.2, CON17.2, US1.2, US1.3, US1.6, US1.7
- new net N$180: CON18.P$1, IC3.1
- new net N$181: CON18.P$2, IC3.2
- new net N$182: CON18.P$3, IC3.3
- new net N$183: CON18.P$4, IC3.4
- new net N$184: CON18.P$5, IC3.5
- new net N$185: CON18.P$6, IC3.6
- new net N$186: CON18.P$7, IC3.7
- new net N$187: CON18.P$8, IC3.8
- new net N$188: CON19.P$1, IC3.9
- new net N$189: CON19.P$2, IC3.10
- new net N$190: CON19.P$3, IC3.11
- new net N$191: CON19.P$4, IC3.12
- new net N$192: CON19.P$5, IC3.13
- new net N$193: CON19.P$6, IC3.14
- new net N$194: CON19.P$7, IC3.15
- new net N$195: CON19.P$8, IC3.16
- new net N$196: CON20.P$1, IC3.17
- new net N$197: CON20.P$2, IC3.18
- new net N$198: CON20.P$3, IC3.19
- new net N$199: CON20.P$4, IC3.20
- new net N$200: CON20.P$5, IC3.21
- new net N$201: CON20.P$6, IC3.22
- new net N$202: CON20.P$7, IC3.23
- new net N$203: CON20.P$8, IC3.24
- new net N$204: CON21.P$1, IC3.25
- new net N$205: CON21.P$2, IC3.26
- new net N$206: CON21.P$3, IC3.27
- new net N$207: CON21.P$4, IC3.28
- new net N$208: CON21.P$5, IC3.29
- new net N$209: CON21.P$6, IC3.30
- new net N$210: CON21.P$7, IC3.31
- new net N$211: CON21.P$8, IC3.32
- new net N$212: C4.1, CON22.1, US2.1
- new net N$213: C3.1, CON22.3, US2.8
- new net N$214: C3.2, C4.2, CON22.2, US2.2, US2.3, US2.6, US2.7
Routing:
- net N$177: track 0.00 -> 6.22 mm
- net N$213: track 0.00 -> 6.22 mm
- net N$178: track 0.00 -> 6.22 mm
- net N$212: track 0.00 -> 6.22 mm
- net N$92: track 0.00 -> 6.09 mm
- net N$124: track 0.00 -> 5.96 mm
- net N$109: track 0.00 -> 5.96 mm
- net N$77: track 0.00 -> 5.96 mm
- net N$93: track 0.00 -> 5.90 mm
- net N$140: track 0.00 -> 5.90 mm
- net N$125: track 0.00 -> 5.90 mm
- net N$108: track 0.00 -> 5.90 mm
- net N$172: track 0.00 -> 5.85 mm
- net N$91: track 0.00 -> 5.80 mm
- net N$165: track 0.00 -> 5.77 mm
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- added copper zone on layer 1, net N$179
- added copper zone on layer 1, net N$214
Other:
- board text added: "1"
- board text added: "11"
- board text added: "12"
- board text added: "16"
- board text added: "17"
- board text added: "20"
- board text added: "22"
- board text added: "23"
- board text added: "24"
- board text added: "25"
- board text added: "28"
- board text added: "32"
- board text added: "33"
- board text added: "34"
- board text added: "36"
- board text added: "4"
- board text added: "40"
- board text added: "44"
- board text added: "48"
- board text added: "49"
- board text added: "52"
- board text added: "56"
- board text added: "60"
- board text added: "64"
- board text added: "8"
- board text added: "9."
- board text added: "GND"
- board text added: "I"
- board text added: "O"

Commit message: Minor corrections. Ready to send.
Parts:
- moved CON11 0.18 mm to (25.6, 35.4)
- moved CON16 0.18 mm to (42.4, 16.4)
- moved CON21 0.18 mm to (26.9, 16.4)
- moved CON7 0.18 mm to (47.5, 38.6)
- moved CON8 0.18 mm to (38.6, 47.5)
- moved U$1 0.18 mm to (38.6, 38.6)
- moved CON10 0.18 mm to (13.8, 23.4)
- moved CON12 0.18 mm to (13.8, 47.5)
- moved CON13 0.18 mm to (37.3, 9.40)
- moved CON15 0.18 mm to (47.5, 9.40)
- moved CON18 0.18 mm to (19.9, 9.40)
- moved CON3 0.18 mm to (16.4, 9.40)
- moved CON4 0.18 mm to (9.40, 16.4)
- moved IC2 0.18 mm to (42.4, 9.40)
- moved IC3 0.18 mm to (26.9, 9.40)
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Other:
- board size 50 x 50 mm -> 49.7 x 49.7 mm
